File: hardware/ir-blaster/ir-blaster.kicad_sch (KiCad schematic)
At the start: 19 parts, among them J1 PWR, J2 DS18B20 [opt], Q1 DMN2046U, U1 ESP32-C3_SUPERMINI

Commit message: added LTSpice sim
Parts:
- C1, C2, C3, C4: value 100nF -> 220nF
- R3, R4, R5: value 33 -> 47
- R7: value 0 -> 1
Other:
- moved on the sheet: C1, C2, C3, C4, D1, D2, D3, J1, J2, Q1, R1, R2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

Commit message: New traces layout
Parts:
- added R9: 4.7k, Resistor_SMD:R_0805_2012Metric_Pad1.20x1.40mm_HandSolder, symbol Device:R_US
- R1: value 270 -> 560
Connections:
- net GND: now also J2.2 (Pin_2), R9.1; no longer J2.1 (Pin_1)
- net IR_OUT: now also U1.1 (GPIO1); no longer U1.7 (GPIO7)
- net at U1.0 (GPIO0): now also J2.1 (Pin_1), R8.1, R9.2
Other:
- moved on the sheet: J1, J2, R8, U1
